File: kicad-project/power.kicad_sch (KiCad schematic)
At the start: 26 parts, among them J3 USB_B_Mini, J4 12V IN, U3 TPS563201

Commit message: hw: classroom changes
Parts:
- R10: Tolerance (none) -> 1%
- renumbered SRP2512-2R2M1 to L1
Changed lines of the file:
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@@
   )
   (symbol (lib_id "Device:R") (at 162.56 57.15 0) (unit 1)
-    (in_bom yes) (on_board yes) (fields_autoplaced)
-    (property "Reference" "R10" (id 0) (at 164.465 55.8799 0)
+    (in_bom yes) (on_board yes)
+    (property "Reference" "R10" (id 0) (at 163.83 54.61 0)
       (effects (font (size 1.27 1.27)) (justify left))
     )
-    (property "Value" "33k" (id 1) (at 164.465 58.4199 0)
+    (property "Value" "33k" (id 1) (at 163.83 57.15 0)
       (effects (font (size 1.27 1.27)) (justify left))
     )
@@
     (property "Datasheet" "~" (id 3) (at 162.56 57.15 0)
       (effects (font (size 1.27 1.27)) hide)
+    )
+    (property "Tolerance" "1%" (id 4) (at 163.83 59.69 0)
+      (effects (font (size 1.27 1.27)) (justify left))
     )
     (pin "1")
@@
   )
   (symbol (lib_id "Device:R") (at 162.56 67.31 0) (unit 1)
-    (in_bom yes) (on_board yes) (fields_autoplaced)
-    (property "Reference" "R11" (id 0) (at 164.465 66.0399 0)
+    (in_bom yes) (on_board yes)
+    (property "Reference" "R11" (id 0) (at 163.83 64.77 0)
       (effects (font (size 1.27 1.27)) (justify left))
     )
-    (property "Value" "10k" (id 1) (at 164.465 68.5799 0)
+    (property "Value" "10k" (id 1) (at 163.83 67.31 0)
       (effects (font (size 1.27 1.27)) (justify left))
     )
@@
   (symbol (lib_id "Device:L") (at 191.77 30.48 90) (unit 1)
     (in_bom yes) (on_board yes) (fields_autoplaced)
-    (property "Reference" "SRP2512-2R2M1" (id 0) (at 191.77 24.13 90))
+    (property "Reference" "L1" (id 0) (at 191.77 24.13 90))
     (property "Value" "2.2u" (id 1) (at 191.77 26.67 90))
     (property "Footprint" "ppse_2021:Inductor" (id 2) (at 191.77 30.48 0)

Commit message: hw: power routing
Connections:
- net 12V_Post_PPTC: now reaches D1.1 (A1), D4.2 (A), F1.1
- net 12V_Post_Fuse: now reaches D2.1 (A1), D3.2 (A), F2.2
Other:
- moved on the sheet: F1, F2, J4
Changed lines of the file:
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@@
   (junction (at 227.33 30.48) (diameter 0) (color 0 0 0 0)
   )
+  (junction (at 41.91 30.48) (diameter 0) (color 0 0 0 0)
+  )
   (junction (at 91.44 50.8) (diameter 0) (color 0 0 0 0)
   )
   (junction (at 209.55 38.1) (diameter 0) (color 0 0 0 0)
-  )
-  (junction (at 52.07 30.48) (diameter 0) (color 0 0 0 0)
   )
   (junction (at 115.57 30.48) (diameter 0) (color 0 0 0 0)
@@
     (stroke (width 0) (type default) (color 0 0 0 0))
   )
+  (wire (pts (xy 41.91 30.48) (xy 46.99 30.48))
+    (stroke (width 0) (type default) (color 0 0 0 0))
+  )
   (wire (pts (xy 45.72 91.44) (xy 53.34 91.44))
     (stroke (width 0) (type default) (color 0 0 0 0))
   )
-  (wire (pts (xy 52.07 30.48) (xy 54.61 30.48))
-    (stroke (width 0) (type default) (color 0 0 0 0))
-  )
   (polyline (pts (xy 114.3 115.57) (xy 27.94 115.57))
     (stroke (width 0) (type default) (color 0 0 0 0))
@@
     (stroke (width 0) (type default) (color 0 0 0 0))
   )
-  (wire (pts (xy 52.07 50.8) (xy 52.07 30.48))
+  (wire (pts (xy 41.91 50.8) (xy 41.91 30.48))
     (stroke (width 0) (type default) (color 0 0 0 0))
   )
@@
     (stroke (width 0) (type default) (color 0 0 0 0))
   )
-  (wire (pts (xy 54.61 50.8) (xy 52.07 50.8))
+  (wire (pts (xy 46.99 50.8) (xy 41.91 50.8))
     (stroke (width 0) (type default) (color 0 0 0 0))
   )
@@
     (stroke (width 0) (type default) (color 0 0 0 0))
   )
-  (wire (pts (xy 62.23 30.48) (xy 69.85 30.48))
-    (stroke (width 0) (type default) (color 0 0 0 0))
-  )
-  (wire (pts (xy 62.23 50.8) (xy 69.85 50.8))
+  (wire (pts (xy 54.61 30.48) (xy 69.85 30.48))
+    (stroke (width 0) (type default) (color 0 0 0 0))
+  )
+  (wire (pts (xy 54.61 50.8) (xy 69.85 50.8))
     (stroke (width 0) (type default) (color 0 0 0 0))
   )
@@
     (stroke (width 0) (type default) (color 0 0 0 0))
   )
-  (wire (pts (xy 45.72 30.48) (xy 52.07 30.48))
+  (wire (pts (xy 33.02 30.48) (xy 41.91 30.48))
     (stroke (width 0) (type default) (color 0 0 0 0))
   )
@@
     (effects (font (size 1.27 1.27)) (justify left bottom))
   )
-  (text "0.5 Hold 1A Trip" (at 53.34 34.29 0)
+  (text "0.5 Hold 1A Trip" (at 45.72 34.29 0)
     (effects (font (size 1.27 1.27)) (justify left bottom))
   )
@@
     (effects (font (size 3 3) (thickness 0.6) bold) (justify left bottom))
   )
-  (text "0.5A per motore" (at 49.53 55.88 0)
+  (text "0.5A per motore" (at 41.91 55.88 0)
     (effects (font (size 1.27 1.27)) (justify left bottom))
   )
@@
     (effects (font (size 1.27 1.27)) (justify left bottom))
   )
-  (label "12V_IN" (at 45.72 30.48 0)
+  (label "12V_IN" (at 33.02 30.48 0)
     (effects (font (size 1.27 1.27)) (justify left bottom))
   )
@@
     (effects (font (size 1.27 1.27)) (justify left bottom))
   )
+  (label "12V_Post_PPTC" (at 58.42 30.48 0)
+    (effects (font (size 1.27 1.27)) (justify left bottom))
+  )
+  (label "12V_Post_Fuse" (at 58.42 50.8 0)
+    (effects (font (size 1.27 1.27)) (justify left bottom))
+  )
   (label "VBUS" (at 46.99 91.44 0)
     (effects (font (size 1.27 1.27)) (justify left bottom))
@@
     (effects (font (size 1.27 1.27)) (justify left))
   )
-  (symbol (lib_id "power:GND") (at 45.72 33.02 0) (unit 1)
-    (in_bom yes) (on_board yes)
-    (property "Reference" "#PWR041" (id 0) (at 45.72 39.37 0)
-      (effects (font (size 1.27 1.27)) hide)
-    )
-    (property "Value" "GND" (id 1) (at 45.847 37.4142 0))
-    (property "Footprint" "" (id 2) (at 45.72 33.02 0)
-      (effects (font (size 1.27 1.27)) hide)
-    )
-    (property "Datasheet" "" (id 3) (at 45.72 33.02 0)
-      (effects (font (size 1.27 1.27)) hide)
-    )
-    (pin "1")
-  )
-  (symbol (lib_id "Device:Polyfuse") (at 58.42 30.48 270) (unit 1)
-    (in_bom yes) (on_board yes)
-    (property "Reference" "F1" (id 0) (at 58.42 24.765 90))
-    (property "Value" "2016L050MR" (id 1) (at 58.42 27.0764 90))
-    (property "Footprint" "ppse_2021:2016L Series PPTC" (id 2) (at 53.34 31.75 0)
+  (symbol (lib_id "power:GND") (at 33.02 33.02 0) (unit 1)
+    (in_bom yes) (on_board yes)
+    (property "Reference" "#PWR041" (id 0) (at 33.02 39.37 0)
+      (effects (font (size 1.27 1.27)) hide)
+    )
+    (property "Value" "GND" (id 1) (at 33.147 37.4142 0))
+    (property "Footprint" "" (id 2) (at 33.02 33.02 0)
+      (effects (font (size 1.27 1.27)) hide)
+    )
+    (property "Datasheet" "" (id 3) (at 33.02 33.02 0)
+      (effects (font (size 1.27 1.27)) hide)
+    )
+    (pin "1")
+  )
+  (symbol (lib_id "Device:Polyfuse") (at 50.8 30.48 270) (unit 1)
+    (in_bom yes) (on_board yes)
+    (property "Reference" "F1" (id 0) (at 50.8 24.765 90))
+    (property "Value" "2016L050MR" (id 1) (at 50.8 27.0764 90))
+    (property "Footprint" "ppse_2021:2016L Series PPTC" (id 2) (at 45.72 31.75 0)
       (effects (font (size 1.27 1.27)) (justify left) hide)
     )
-    (property "Datasheet" "https://www.farnell.com/datasheets/664999.pdf" (id 3) (at 58.42 30.48 0)
+    (property "Datasheet" "https://www.farnell.com/datasheets/664999.pdf" (id 3) (at 50.8 30.48 0)
       (effects (font (size 1.27 1.27)) hide)
     )
@@
     (pin "1")
   )
-  (symbol (lib_id "Connector_Generic:Conn_01x02") (at 40.64 33.02 180) (unit 1)
-    (in_bom yes) (on_board yes) (fields_autoplaced)
-    (property "Reference" "J4" (id 0) (at 40.64 24.13 0))
-    (property "Value" "12V IN" (id 1) (at 40.64 26.67 0))
-    (property "Footprint" "Connector_Molex:Molex_Micro-Fit_3.0_43650-0200_1x02_P3.00mm_Horizontal" (id 2) (at 40.64 33.02 0)
-      (effects (font (size 1.27 1.27)) hide)
-    )
-    (property "Datasheet" "~" (id 3) (at 40.64 33.02 0)
+  (symbol (lib_id "Connector_Generic:Conn_01x02") (at 27.94 33.02 180) (unit 1)
+    (in_bom yes) (on_board yes) (fields_autoplaced)
+    (property "Reference" "J4" (id 0) (at 27.94 24.13 0))
+    (property "Value" "12V IN" (id 1) (at 27.94 26.67 0))
+    (property "Footprint" "Connector_Molex:Molex_Micro-Fit_3.0_43650-0200_1x02_P3.00mm_Horizontal" (id 2) (at 27.94 33.02 0)
+      (effects (font (size 1.27 1.27)) hide)
+    )
+    (property "Datasheet" "~" (id 3) (at 27.94 33.02 0)
       (effects (font (size 1.27 1.27)) hide)
     )
@@
     (pin "1")
   )
-  (symbol (lib_id "Device:Fuse") (at 58.42 50.8 90) (unit 1)
-    (in_bom yes) (on_board yes) (fields_autoplaced)
-    (property "Reference" "F2" (id 0) (at 58.42 44.45 90))
-    (property "Value" "Fuse 1.5A" (id 1) (at 58.42 46.99 90))
-    (property "Footprint" "ppse_2021:Fuse Holder" (id 2) (at 58.42 52.578 90)
-      (effects (font (size 1.27 1.27)) hide)
-    )
-    (property "Datasheet" "https://www.farnell.com/datasheets/2074958.pdf" (id 3) (at 58.42 50.8 0)
-      (effects (font (size 1.27 1.27)) hide)
-    )
+  (symbol (lib_id "Device:Fuse") (at 50.8 50.8 90) (unit 1)
+    (in_bom yes) (on_board yes) (fields_autoplaced)
+    (property "Reference" "F2" (id 0) (at 50.8 44.45 90))
+    (property "Value" "Fuse 1.5A" (id 1) (at 50.8 46.99 90))
+    (property "Footprint" "ppse_2021:Fuse Holder" (id 2) (at 50.8 52.578 90)
+      (effects (font (size 1.27 1.27)) hide)
+    )
+    (property "Datasheet" "https://www.farnell.com/datasheets/2074958.pdf" (id 3) (at 50.8 50.8 0)
+      (effects (font (size 1.27 1.27)) hide)
+    )
