File: kicad-project/connectivity.kicad_sch (KiCad schematic)
At the start: 21 parts, among them J5 Compass, J6 Accelerometer, J7 OLED, Q1 3LP01M, Q2 PDTC114Y, Q3 BC846A, Q4 BC846A, Q5 BC846A, U4 PAM-7Q-0

Commit message: hw: final changes
Connections:
- net GND: now also U4.MP1, U4.MP2
- no-connect marks 6 -> 4
Changed lines of the file:
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@@
   (no_connect (at 191.77 133.35))
   (no_connect (at 99.06 59.69))
-  (no_connect (at 118.11 72.39))
-  (no_connect (at 115.57 72.39))
   (polyline (pts (xy 157.48 13.97) (xy 157.48 82.55))
     (stroke (width 0) (type default) (color 0 0 0 0))
@@
     (pin "MP2")
   )
+  (symbol (lib_id "power:GND") (at 115.57 72.39 0) (unit 1)
+    (in_bom yes) (on_board yes)
+    (property "Reference" "#PWR?" (id 0) (at 115.57 78.74 0)
+      (effects (font (size 1.27 1.27)) hide)
+    )
+    (property "Value" "GND" (id 1) (at 115.57 77.47 90))
+    (property "Footprint" "" (id 2) (at 115.57 72.39 0)
+      (effects (font (size 1.27 1.27)) hide)
+    )
+    (property "Datasheet" "" (id 3) (at 115.57 72.39 0)
+      (effects (font (size 1.27 1.27)) hide)
+    )
+    (pin "1")
+  )
   (symbol (lib_id "Connector_Generic:Conn_01x05") (at 196.85 104.14 0) (unit 1)
     (in_bom yes) (on_board yes) (fields_autoplaced)
@@
     (pin "2")
   )
+  (symbol (lib_id "power:GND") (at 118.11 72.39 0) (unit 1)
+    (in_bom yes) (on_board yes)
+    (property "Reference" "#PWR?" (id 0) (at 118.11 78.74 0)
+      (effects (font (size 1.27 1.27)) hide)
+    )
+    (property "Value" "GND" (id 1) (at 118.11 77.47 90))
+    (property "Footprint" "" (id 2) (at 118.11 72.39 0)
+      (effects (font (size 1.27 1.27)) hide)
+    )
+    (property "Datasheet" "" (id 3) (at 118.11 72.39 0)
+      (effects (font (size 1.27 1.27)) hide)
+    )
+    (pin "1")
+  )
   (symbol (lib_id "Device:R") (at 49.53 110.49 0) (unit 1)

Commit message: hw: add custom page layout
Other:
- company: Connectivity -> (none)
- title: (none) -> Peripherals
Changed lines of the file:
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@@
   (paper "A4")
   (title_block
-    (company "Connectivity")
+    (title "Peripherals")
+    (date "2022-04-13")
+    (rev "1.0")
   )
   (junction (at 49.53 105.41) (diameter 0) (color 0 0 0 0)

Commit message: hw: changes for the simia
Parts:
- D7: value LED_RGB 5050 -> LED_RGB 1210
Connections:
- net GPS_EN renamed ~{GPS_EN}
Other:
- note added: "Accelerometer"
- note added: "Magnetometer"
- note removed: "occhio ai pin nel footprint del led RGB"
- moved on the sheet: BZ1, C24, C25, D7, J5, J6, J7, Q1, Q2, Q3, Q4, Q5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
